Commit message: fix: rename joint for consistency in xacro definition

File: urdf/abb_irbt4004_macro.xacro (robot description, xacro)
@@ -74,5 +74,5 @@
         <origin xyz="0 0 0" rpy="0 0 0"/>
     </joint>
-    <joint name="${prefix}ext_1" type="prismatic">
+    <joint name="joint_${prefix}ext_1" type="prismatic">
       <parent link="${prefix}track"/>
       <child link="${prefix}carriage"/>
